File: levelhacker.sch (KiCad schematic (older format))
At the start: 26 parts, among them IC1 ATTINY1634-SU, P1 PROGRAMMING_HEADER, U1 MMA8652

Commit message: Add footprints for the RGB leds
Parts:
- D1, D2, D3, D4: footprint (none) -> workshop-footprints:LED_LUMEXLXT0805
Changed lines of the file:
@@
 F 0 "D2" H 5650 4165 50  0000 C CNN
 F 1 "LED_RGB2" H 5650 4074 50  0000 C CNN
-F 2 "" H 5600 3650 50  0000 C CNN
+F 2 "workshop-footprints:LED_LUMEXLXT0805" H 5600 3650 50  0001 C CNN
 F 3 "" H 5600 3650 50  0000 C CNN
 	1    5650 3700
@@
 F 0 "D3" H 6450 3265 50  0000 C CNN
 F 1 "LED_RGB3" H 6450 3174 50  0000 C CNN
-F 2 "" H 6400 2750 50  0000 C CNN
+F 2 "workshop-footprints:LED_LUMEXLXT0805" H 6400 2750 50  0001 C CNN
 F 3 "" H 6400 2750 50  0000 C CNN
 	1    6450 2800
@@
 F 0 "D1" H 5650 3265 50  0000 C CNN
 F 1 "LED_RGB1" H 5650 3174 50  0000 C CNN
-F 2 "" H 5600 2750 50  0000 C CNN
+F 2 "workshop-footprints:LED_LUMEXLXT0805" H 5600 2750 50  0001 C CNN
 F 3 "" H 5600 2750 50  0000 C CNN
 	1    5650 2800
@@
 F 0 "D4" H 6450 4165 50  0000 C CNN
 F 1 "LED_RGB4" H 6450 4074 50  0000 C CNN
-F 2 "" H 6400 3650 50  0000 C CNN
+F 2 "workshop-footprints:LED_LUMEXLXT0805" H 6400 3650 50  0001 C CNN
 F 3 "" H 6400 3650 50  0000 C CNN
 	1    6450 3700

Commit message: Add footprints for the coin cell battery and accel.
Parts:
- BT1: footprint (none) -> workshop-footprints:battery-2032
- C1, C2, C3, C4: footprint (none) -> Capacitors_SMD:C_1206
- IC1: footprint SO20 -> Housings_SOIC:SOIC-20W_7.5x12.8mm_Pitch1.27mm
- P1: footprint (none) -> Pin_Headers:Pin_Header_Straight_SMT_02x03
- R1, R10, R11, R12, R13, R14, R2, R3, R4, R5, R6, R7, R8, R9: footprint (none) -> Resistors_SMD:R_1206
- U1: footprint (none) -> workshop-footprints:DFN-10-1EP_2x2mm_Pitch0.4mm
Changed lines of the file:
@@
 F 0 "IC1" H 2800 4707 50  0000 C CNN
 F 1 "ATTINY1634-SU" H 2800 4616 50  0000 C CNN
-F 2 "SO20" H 2800 4525 50  0000 C CIN
+F 2 "Housings_SOIC:SOIC-20W_7.5x12.8mm_Pitch1.27mm" H 2800 4525 50  0000 C CIN
 F 3 "" H 2800 3750 50  0000 C CNN
 	1    2800 3300
@@
 F 0 "P1" H 2450 5365 50  0000 C CNN
 F 1 "PROGRAMMING_HEADER" H 2450 5274 50  0000 C CNN
-F 2 "" H 2450 3850 50  0000 C CNN
+F 2 "Pin_Headers:Pin_Header_Straight_SMT_02x03" H 2450 3850 50  0001 C CNN
 F 3 "" H 2450 3850 50  0000 C CNN
 	1    2450 5050
@@
 F 0 "U1" H 2850 1987 60  0000 C CNN
 F 1 "MMA8652" H 2850 1881 60  0000 C CNN
-F 2 "" H 2850 1450 60  0001 C CNN
+F 2 "workshop-footprints:DFN-10-1EP_2x2mm_Pitch0.4mm" H 2850 1450 60  0001 C CNN
 F 3 "" H 2850 1450 60  0001 C CNN
 	1    2850 1450
@@
 F 0 "C1" H 1741 1396 50  0000 L CNN
 F 1 "1uf" H 1741 1305 50  0000 L CNN
-F 2 "" H 1650 1350 50  0000 C CNN
+F 2 "Capacitors_SMD:C_1206" H 1650 1350 50  0001 C CNN
 F 3 "" H 1650 1350 50  0000 C CNN
 	1    1650 1350
@@
 F 0 "C2" H 1708 1304 50  0000 R CNN
 F 1 ".1uf" H 1708 1395 50  0000 R CNN
-F 2 "" H 1800 1350 50  0000 C CNN
+F 2 "Capacitors_SMD:C_1206" H 1800 1350 50  0001 C CNN
 F 3 "" H 1800 1350 50  0000 C CNN
 	1    1800 1350
@@
 F 0 "C3" H 2391 1696 50  0000 L CNN
 F 1 ".1uf" H 2391 1605 50  0000 L CNN
-F 2 "" H 2300 1650 50  0000 C CNN
+F 2 "Capacitors_SMD:C_1206" H 2300 1650 50  0001 C CNN
 F 3 "" H 2300 1650 50  0000 C CNN
 	1    2300 1650
@@
 F 0 "R1" H 4009 2196 50  0000 L CNN
 F 1 "10k" H 4009 2105 50  0000 L CNN
-F 2 "" H 3950 2150 50  0000 C CNN
+F 2 "Resistors_SMD:R_1206" H 3950 2150 50  0001 C CNN
 F 3 "" H 3950 2150 50  0000 C CNN
 	1    3950 2150
@@
 F 0 "R2" V 5346 2500 50  0000 C CNN
 F 1 "R_Small" V 5255 2500 50  0000 C CNN
-F 2 "" H 5150 2500 50  0000 C CNN
+F 2 "Resistors_SMD:R_1206" H 5150 2500 50  0001 C CNN
 F 3 "" H 5150 2500 50  0000 C CNN
 	1    5150 2500
@@
 F 0 "R3" V 5346 2800 50  0000 C CNN
 F 1 "R_Small" V 5255 2800 50  0000 C CNN
-F 2 "" H 5150 2800 50  0000 C CNN
+F 2 "Resistors_SMD:R_1206" H 5150 2800 50  0001 C CNN
 F 3 "" H 5150 2800 50  0000 C CNN
 	1    5150 2800
@@
 F 0 "R4" V 5346 3100 50  0000 C CNN
 F 1 "R_Small" V 5255 3100 50  0000 C CNN
-F 2 "" H 5150 3100 50  0000 C CNN
+F 2 "Resistors_SMD:R_1206" H 5150 3100 50  0001 C CNN
 F 3 "" H 5150 3100 50  0000 C CNN
 	1    5150 3100
@@
 F 0 "R8" V 7146 2500 50  0000 C CNN
 F 1 "R_Small" V 7055 2500 50  0000 C CNN
-F 2 "" H 6950 2500 50  0000 C CNN
+F 2 "Resistors_SMD:R_1206" H 6950 2500 50  0001 C CNN
 F 3 "" H 6950 2500 50  0000 C CNN
 	1    6950 2500
@@
 F 0 "R9" V 7146 2800 50  0000 C CNN
 F 1 "R_Small" V 7055 2800 50  0000 C CNN
-F 2 "" H 6950 2800 50  0000 C CNN
+F 2 "Resistors_SMD:R_1206" H 6950 2800 50  0001 C CNN
 F 3 "" H 6950 2800 50  0000 C CNN
 	1    6950 2800
@@
 F 0 "R10" V 7146 3100 50  0000 C CNN
 F 1 "R_Small" V 7055 3100 50  0000 C CNN
-F 2 "" H 6950 3100 50  0000 C CNN
+F 2 "Resistors_SMD:R_1206" H 6950 3100 50  0001 C CNN
 F 3 "" H 6950 3100 50  0000 C CNN
 	1    6950 3100
@@
 F 0 "R5" V 5346 3400 50  0000 C CNN
 F 1 "R_Small" V 5255 3400 50  0000 C CNN
-F 2 "" H 5150 3400 50  0000 C CNN
+F 2 "Resistors_SMD:R_1206" H 5150 3400 50  0001 C CNN
 F 3 "" H 5150 3400 50  0000 C CNN
 	1    5150 3400
@@
 F 0 "R6" V 5346 3700 50  0000 C CNN
 F 1 "R_Small" V 5255 3700 50  0000 C CNN
-F 2 "" H 5150 3700 50  0000 C CNN
+F 2 "Resistors_SMD:R_1206" H 5150 3700 50  0001 C CNN
 F 3 "" H 5150 3700 50  0000 C CNN
 	1    5150 3700
@@
 F 0 "R7" V 5346 4000 50  0000 C CNN
 F 1 "R_Small" V 5255 4000 50  0000 C CNN
-F 2 "" H 5150 4000 50  0000 C CNN
+F 2 "Resistors_SMD:R_1206" H 5150 4000 50  0001 C CNN
 F 3 "" H 5150 4000 50  0000 C CNN
 	1    5150 4000
@@
 F 0 "R11" V 7146 3400 50  0000 C CNN
 F 1 "R_Small" V 7055 3400 50  0000 C CNN
-F 2 "" H 6950 3400 50  0000 C CNN
+F 2 "Resistors_SMD:R_1206" H 6950 3400 50  0001 C CNN
 F 3 "" H 6950 3400 50  0000 C CNN
 	1    6950 3400
@@
 F 0 "R12" V 7146 3700 50  0000 C CNN
 F 1 "R_Small" V 7055 3700 50  0000 C CNN
-F 2 "" H 6950 3700 50  0000 C CNN
+F 2 "Resistors_SMD:R_1206" H 6950 3700 50  0001 C CNN
 F 3 "" H 6950 3700 50  0000 C CNN
 	1    6950 3700
@@
 F 0 "R13" V 7146 4000 50  0000 C CNN
 F 1 "R_Small" V 7055 4000 50  0000 C CNN
-F 2 "" H 6950 4000 50  0000 C CNN
+F 2 "Resistors_SMD:R_1206" H 6950 4000 50  0001 C CNN
 F 3 "" H 6950 4000 50  0000 C CNN
 	1    6950 4000
@@
 F 0 "C4" H 3791 1596 50  0000 L CNN
 F 1 ".1uf" H 3791 1505 50  0000 L CNN
-F 2 "" H 3700 1550 50  0000 C CNN
+F 2 "Capacitors_SMD:C_1206" H 3700 1550 50  0001 C CNN
 F 3 "" H 3700 1550 50  0000 C CNN
 	1    3700 1550
@@
 F 0 "BT1" H 1018 1896 50  0000 L CNN
 F 1 "Battery" H 1018 1805 50  0000 L CNN
-F 2 "" V 900 1890 50  0000 C CNN
+F 2 "workshop-footprints:battery-2032" V 900 1890 50  0001 C CNN
 F 3 "" V 900 1890 50  0000 C CNN
 	1    900  1850
@@
 F 0 "R14" H 3859 4296 50  0000 L CNN
 F 1 "10k" H 3859 4205 50  0000 L CNN
-F 2 "" H 3800 4250 50  0000 C CNN
+F 2 "Resistors_SMD:R_1206" H 3800 4250 50  0001 C CNN
 F 3 "" H 3800 4250 50  0000 C CNN
 	1    3800 4250
